File: zorionx_nivara/relay.kicad_sch (KiCad schematic)
At the start: 0 parts

Commit message: driver relay
Parts:
- added D2, D3: M7, PCM_Diode_SMD_AKL:D_SMA, symbol PCM_Diode_AKL:M7
- added IC1: BTS723GW, SOIC127P600X175-14N, symbol Samacsys:BTS723GW
- added K1, K2: G6RL-1_DC24, G6RL1DC24, symbol Samacsys:G6RL-1_DC24
Connections:
- new net: D3.1 (K), IC1.10 (OUT2_2), IC1.9 (OUT2_1), K2.1 (COIL_1)
- new net: D2.1 (K), IC1.12 (OUT1_1), IC1.13 (OUT1_2), K1.1 (COIL_1)
- new net GND: D2.2 (A), D3.2 (A), IC1.4 (GND), K1.5 (COIL_2), K2.5 (COIL_2)
- new net RELAY_1_IN: IC1.2 (IN1)
- new net RELAY_2_IN: IC1.6 (IN2)
- new net RLY1_C: K1.2 (COM)
- new net RLY1_NC: K1.4 (NC)
- new net RLY1_NO: K1.3 (NO)
- new net RLY2_C: K2.2 (COM)
- new net RLY2_NC: K2.4 (NC)
- new net RLY2_NO: K2.3 (NO)
- new net VCC: IC1.1 (VBB_1), IC1.14 (VBB_4), IC1.7 (VBB_2), IC1.8 (VBB_3)
