File: zorionx_nivara/zorionx_nivara.kicad_pcb (KiCad board)
At the start: 4 copper layers, 103.1 x 83.7 mm, 25 parts, among them J1 Screw_Terminal_01x02, J2 Screw_Terminal_01x04, J3 Screw_Terminal_01x04, J4 Screw_Terminal_01x02, J5 Screw_Terminal_01x02, J6 Screw_Terminal_01x03, J7 Screw_Terminal_01x04, J8 Screw_Terminal_01x03, J9 Screw_Terminal_01x06, U1 ESP32-S3-WROOM-1, U2 AP63203WU

Commit message: driver relay
Parts:
- added D1: SM712_SOT23, Package_TO_SOT_SMD:SOT-23, F.Cu at (147.7, 120.5)
- added D2: M7, PCM_Diode_SMD_AKL:D_SMA, B.Cu at (108.7, 56.9)
- added D3: M7, PCM_Diode_SMD_AKL:D_SMA, B.Cu at (95.0, 56.4)
- added IC1: BTS723GW, Samacsys:SOIC127P600X175-14N, F.Cu at (120.9, 53.8)
- added K1: G6RL-1_DC24, Samacsys:G6RL1DC24, F.Cu at (112.0, 60.8)
- added K2: G6RL-1_DC24, Samacsys:G6RL1DC24, F.Cu at (98.8, 60.8)
Routing:
- net /board_zorionx-nivara/RLY1_NC: track 0.00 -> 19.9 mm
- net /board_zorionx-nivara/RLY2_NC: track 0.00 -> 19.1 mm
- net /board_zorionx-nivara/RLY1_C: track 0.00 -> 15.7 mm
- net /board_zorionx-nivara/RLY2_C: track 0.00 -> 14.8 mm
- net /board_zorionx-nivara/RLY1_NO: track 0.00 -> 11.4 mm
- net /board_zorionx-nivara/RLY2_NO: track 0.00 -> 10.6 mm
